Commit message: made beacon cameras look slightly downward

File: src/nucobot_simulator/nucobot_description/urdf/tower.xacro (robot description, xacro)
@@ -33,5 +33,5 @@
     <parent link="tower_$(arg prefix)_base_link"/>
     <child link="tower_$(arg prefix)_camera_link"/>
-    <origin xyz="${width} ${width/2} ${height}" rpy="0 0 0"/>
+    <origin xyz="${width} ${width/2} ${height}" rpy="0 0.5 0"/>
   </joint>
   <link name="tower_$(arg prefix)_camera_link">
