Commit message: - renamed the tower model to 'beacon' and moved it to separate folder  - started working on the addition of game elements (cylinders, cups, etc.)

File: src/nucobot_simulator/nucobot_description/urdf/beacon/beacon.xacro (robot description, xacro)
@@ -1,4 +1,4 @@
 <?xml version="1.0"?>
-<robot name="tower_$(arg prefix)" xmlns:xacro="http://www.ros.org/wiki/xacro">
+<robot name="beacon_$(arg prefix)" xmlns:xacro="http://www.ros.org/wiki/xacro">
   <!-- Constants for robot dimensions -->
   <xacro:property name="PI" value="3.1415926535897931"/>
@@ -6,9 +6,9 @@
   <xacro:property name="height" value="0.16" />
   <!-- Import all Gazebo-customization elements, including Gazebo colors -->
-  <xacro:include filename="$(find nucobot_description)/urdf/tower.gazebo" />
+  <xacro:include filename="$(find nucobot_description)/urdf/beacon/beacon.gazebo" />
   <!-- Import Rviz colors -->
   <xacro:include filename="$(find nucobot_description)/urdf/materials.xacro" />
   <!-- Camera -->
-  <link name="tower_$(arg prefix)_base_link">
+  <link name="beacon_$(arg prefix)_base_link">
     <collision>
       <origin xyz="0 0 ${height/2}" rpy="0 0 0"/>
@@ -30,10 +30,10 @@
     </inertial>
   </link>
-  <joint name="tower_$(arg prefix)_base_to_camera" type="fixed">
-    <parent link="tower_$(arg prefix)_base_link"/>
-    <child link="tower_$(arg prefix)_camera_link"/>
+  <joint name="beacon_$(arg prefix)_base_to_camera" type="fixed">
+    <parent link="beacon_$(arg prefix)_base_link"/>
+    <child link="beacon_$(arg prefix)_camera_link"/>
     <origin xyz="${width} ${width/2} ${height}" rpy="0 0.5 0"/>
   </joint>
-  <link name="tower_$(arg prefix)_camera_link">
+  <link name="beacon_$(arg prefix)_camera_link">
     <inertial>
       <mass value="1e-6" />
