Commit message: added cup, tennis ball, pop corn ball and fixed cylinder models; still using turtlebot as a robot

File: src/nucobot_simulator/nucobot_description/urdf/toys/cup.xacro (robot description, xacro)
@@ -1,14 +1,14 @@
 <?xml version="1.0"?>
-<robot name="cylinder_$(arg prefix)" xmlns:xacro="http://www.ros.org/wiki/xacro">
-  <gazebo reference="cylinder_$(arg prefix)_base_link">
+<robot name="cup_$(arg prefix)" xmlns:xacro="http://www.ros.org/wiki/xacro">
+  <gazebo reference="cup_$(arg prefix)_base_link">
     <mu1>0.2</mu1>
     <mu2>0.2</mu2>
     <material>Gazebo/White</material>
   </gazebo>
-  <link name="cylinder_$(arg prefix)_base_link">
+  <link name="cup_$(arg prefix)_base_link">
     <collision>
       <origin xyz="0 0 0" rpy="0 0 0"/>
       <geometry>
-        <mesh filename="package://nucobot_description/meshes/toys/cylinder.dae"/>
+        <mesh filename="package://nucobot_description/meshes/toys/cup.dae"/>
       </geometry>
     </collision>
@@ -16,5 +16,5 @@
       <origin xyz="0 0 0" rpy="0 0 0"/>
       <geometry>
-        <mesh filename="package://nucobot_description/meshes/toys/cylinder.dae"/>
+        <mesh filename="package://nucobot_description/meshes/toys/cup.dae"/>
       </geometry>
     </visual>

File: src/nucobot_simulator/nucobot_description/urdf/toys/pop_corn_ball.xacro (robot description, xacro)
@@ -1,14 +1,13 @@
 <?xml version="1.0"?>
-<robot name="cylinder_$(arg prefix)" xmlns:xacro="http://www.ros.org/wiki/xacro">
-  <gazebo reference="cylinder_$(arg prefix)_base_link">
+<robot name="pop_corn_ball_$(arg prefix)" xmlns:xacro="http://www.ros.org/wiki/xacro">
+  <gazebo reference="pop_corn_ball_$(arg prefix)_base_link">
     <mu1>0.2</mu1>
     <mu2>0.2</mu2>
-    <material>Gazebo/White</material>
   </gazebo>
-  <link name="cylinder_$(arg prefix)_base_link">
+  <link name="pop_corn_ball_$(arg prefix)_base_link">
     <collision>
       <origin xyz="0 0 0" rpy="0 0 0"/>
       <geometry>
-        <mesh filename="package://nucobot_description/meshes/toys/cylinder.dae"/>
+        <mesh filename="package://nucobot_description/meshes/toys/pop_corn_ball.dae"/>
       </geometry>
     </collision>
@@ -16,5 +15,5 @@
       <origin xyz="0 0 0" rpy="0 0 0"/>
       <geometry>
-        <mesh filename="package://nucobot_description/meshes/toys/cylinder.dae"/>
+        <mesh filename="package://nucobot_description/meshes/toys/pop_corn_ball.dae"/>
       </geometry>
     </visual>

File: src/nucobot_simulator/nucobot_description/urdf/toys/tennis_ball.xacro (robot description, xacro)
@@ -1,14 +1,13 @@
 <?xml version="1.0"?>
-<robot name="cylinder_$(arg prefix)" xmlns:xacro="http://www.ros.org/wiki/xacro">
-  <gazebo reference="cylinder_$(arg prefix)_base_link">
+<robot name="tennis_ball_$(arg prefix)" xmlns:xacro="http://www.ros.org/wiki/xacro">
+  <gazebo reference="tennis_ball_$(arg prefix)_base_link">
     <mu1>0.2</mu1>
     <mu2>0.2</mu2>
-    <material>Gazebo/White</material>
   </gazebo>
-  <link name="cylinder_$(arg prefix)_base_link">
+  <link name="tennis_ball_$(arg prefix)_base_link">
     <collision>
       <origin xyz="0 0 0" rpy="0 0 0"/>
       <geometry>
-        <mesh filename="package://nucobot_description/meshes/toys/cylinder.dae"/>
+        <mesh filename="package://nucobot_description/meshes/toys/tennis_ball.dae"/>
       </geometry>
     </collision>
@@ -16,5 +15,5 @@
       <origin xyz="0 0 0" rpy="0 0 0"/>
       <geometry>
-        <mesh filename="package://nucobot_description/meshes/toys/cylinder.dae"/>
+        <mesh filename="package://nucobot_description/meshes/toys/tennis_ball.dae"/>
       </geometry>
     </visual>
