Commit message: - changed 'world' frame to 'map'; configured gmapping on a 'test_base' platform

File: src/nucobot_simulator/nucobot_description/urdf/test_base/test_base_kinect.urdf.xacro (robot description, xacro)
@@ -1,16 +1,7 @@
 <?xml version="1.0"?>
-<robot name="nucobot" xmlns:xacro="http://www.ros.org/wiki/xacro">
+<robot name="test_base_kinect" xmlns:xacro="http://www.ros.org/wiki/xacro">
   <xacro:include filename="$(find nucobot_description)/urdf/materials.xacro" />
   <property name="M_PI" value="3.1415926535897931" />
   <link name="base_footprint"/>
-  <!--
-     Base link is set at the bottom of the base mould.
-     This is done to be compatible with the way base link
-     was configured for turtlebot 1. Refer to
-     https://github.com/turtlebot/turtlebot/issues/40
-     To put the base link at the more oft used wheel
-     axis, set the z-distance from the base_footprint
-     to 0.352.
-    -->
   <joint name="base_joint" type="fixed">
     <origin xyz="0 0 0.0102" rpy="0 0 0" />
@@ -39,9 +30,8 @@
     </inertial>
   </link>
-  <joint name="wheel_left_joint" type="continuous">
+  <joint name="wheel_left_joint" type="fixed">
     <parent link="base_link"/>
     <child link="wheel_left_link"/>
     <origin xyz="0.00 ${0.23/2} 0.0250" rpy="${-M_PI/2} 0 0"/>
-    <axis xyz="0 0 1"/>
   </joint>
   <link name="wheel_left_link">
@@ -66,9 +56,8 @@
     </inertial>
   </link>
-  <joint name="wheel_right_joint" type="continuous">
+  <joint name="wheel_right_joint" type="fixed">
     <parent link="base_link"/>
     <child link="wheel_right_link"/>
     <origin xyz="0.00 -${0.23/2} 0.0250" rpy="${-M_PI/2} 0 0"/>
-    <axis xyz="0 0 1"/>
   </joint>
   <link name="wheel_right_link">
@@ -176,5 +165,5 @@
       <commandTopic>cmd_vel</commandTopic>
       <odometryTopic>odom</odometryTopic>
-      <odometryFrame>odom</odometryFrame>
+      <odometryFrame>world</odometryFrame>
       <robotBaseFrame>base_footprint</robotBaseFrame>
     </plugin>
