Commit message: New robot size + genstatic map was removed

File: src/nucobot_simulator/nucobot_description/urdf/nucobot-2/nucobot.urdf.xacro (robot description, xacro)
@@ -21,5 +21,5 @@
     <visual>
       <geometry>
-        <cylinder length="0.10938" radius="0.178"/>
+        <cylinder length="0.10938" radius="0.15"/>
       </geometry>
       <origin xyz="0.001 0 0.05199" rpy="0 0 0"/>
@@ -27,5 +27,5 @@
     <collision>
       <geometry>
-        <cylinder length="0.10938" radius="0.178"/>
+        <cylinder length="0.10938" radius="0.15"/>
       </geometry>
       <origin xyz="0.0 0 0.05949" rpy="0 0 0"/>
@@ -183,5 +183,5 @@
   <xacro:include filename="$(find nucobot_description)/urdf/sensors/kinect_camera.urdf.xacro" />
   <xacro:kinect_camera name="kinect" parent="base_link">
-    <origin xyz="${0.178/2} 0 ${0.3/2}" rpy="0.0 0.0 0.0"/>
+    <origin xyz="${0.15/2} 0 ${0.3/2}" rpy="0.0 0.0 0.0"/>
   </xacro:kinect_camera>
   <!-- Generic camera

Commit message: add kind of manipulator

File: src/nucobot_simulator/nucobot_description/urdf/nucobot-2/nucobot.urdf.xacro (robot description, xacro)
@@ -3,14 +3,6 @@
   <xacro:include filename="$(find nucobot_description)/urdf/materials.xacro" />
   <property name="M_PI" value="3.1415926535897931" />
+  <property name="RADIUS" value="0.15" />
   <link name="base_footprint"/>
-  <!--
-     Base link is set at the bottom of the base mould.
-     This is done to be compatible with the way base link
-     was configured for turtlebot 1. Refer to
-     https://github.com/turtlebot/turtlebot/issues/40
-     To put the base link at the more oft used wheel
-     axis, set the z-distance from the base_footprint
-     to 0.352.
-    -->
   <joint name="base_joint" type="fixed">
     <origin xyz="0 0 0.0102" rpy="0 0 0" />
@@ -21,5 +13,5 @@
     <visual>
       <geometry>
-        <cylinder length="0.10938" radius="0.15"/>
+        <cylinder length="0.10938" radius="${RADIUS}"/>
       </geometry>
       <origin xyz="0.001 0 0.05199" rpy="0 0 0"/>
@@ -27,5 +19,5 @@
     <collision>
       <geometry>
-        <cylinder length="0.10938" radius="0.15"/>
+        <cylinder length="0.10938" radius="${RADIUS}"/>
       </geometry>
       <origin xyz="0.0 0 0.05949" rpy="0 0 0"/>
@@ -39,4 +31,56 @@
     </inertial>
   </link>
+  <link name="whisker_left">
+    <visual>
+      <geometry>
+        <box size="0.4 0.02 0.02"/>
+      </geometry>
+      <origin xyz="0 0 0" rpy="0 0 0"/>
+    </visual>
+    <collision>
+      <geometry>
+        <box size="0.4 0.02 0.02"/>
+      </geometry>
+      <origin xyz="0 0 0" rpy="0 0 0"/>
+    </collision>
+    <inertial>
+      <origin xyz="0 0 0"/>
+      <mass value="0.4"/>
+      <inertia ixx="0.019995" ixy="0.0" ixz="0.0"
+               iyy="0.019995" iyz="0.0"
+               izz="0.03675" />
+    </inertial>
+  </link>
+  <link name="whisker_right">
+    <visual>
+      <geometry>
+        <box size="0.4 0.02 0.02"/>
+      </geometry>
+      <origin xyz="0 0 0" rpy="0 0 0"/>
+    </visual>
+    <collision>
+      <geometry>
+        <box size="0.4 0.02 0.02"/>
+      </geometry>
+      <origin xyz="0 0 0" rpy="0 0 0"/>
+    </collision>
+    <inertial>
+      <origin xyz="0 0 0"/>
+      <mass value="0.4"/>
+      <inertia ixx="0.019995" ixy="0.0" ixz="0.0"
+               iyy="0.019995" iyz="0.0"
+               izz="0.03675" />
+    </inertial>
+  </link>
+  <joint name="base2whisker_l" type="fixed">
+    <origin xyz="${RADIUS} ${RADIUS/3} ${RADIUS/2}" rpy="0 0 ${M_PI/6}" />
+    <parent link="base_link"/>
+    <child link="whisker_left" />
+  </joint>
+  <joint name="base2whisker_r" type="fixed">
+    <origin xyz="${RADIUS} ${-RADIUS/3} ${RADIUS/2}" rpy="0 0 ${-M_PI/6}" />
+    <parent link="base_link"/>
+    <child link="whisker_right" />
+  </joint>
   <joint name="wheel_left_joint" type="continuous">
     <parent link="base_link"/>
@@ -183,5 +227,5 @@
   <xacro:include filename="$(find nucobot_description)/urdf/sensors/kinect_camera.urdf.xacro" />
   <xacro:kinect_camera name="kinect" parent="base_link">
-    <origin xyz="${0.15/2} 0 ${0.3/2}" rpy="0.0 0.0 0.0"/>
+    <origin xyz="${RADIUS/2} 0 ${0.3/2}" rpy="0.0 0.0 0.0"/>
   </xacro:kinect_camera>
   <!-- Generic camera
