Commit message: added 'pikea' robot; added 3d models for 'bertha' and 'pikea'

File: src/nucobot_simulator/nucobot_description/urdf/pikea/pikea.urdf.xacro (robot description, xacro)
@@ -1,7 +1,10 @@
 <?xml version="1.0"?>
-<robot name="bertha" xmlns:xacro="http://www.ros.org/wiki/xacro">
+<robot name="pikea" xmlns:xacro="http://www.ros.org/wiki/xacro">
   <xacro:include filename="$(find nucobot_description)/urdf/materials.xacro" />
   <property name="M_PI" value="3.1415926535897931" />
-  <property name="RADIUS" value="0.15" />
+  <property name="WHEEL_SEP" value="0.15" />
+  <property name="WHEEL_DIA" value="0.07" />
+  <property name="WHEEL_HGT" value="-0.08" />
+  <property name="WHEEL_SHIFT" value="-0.02" />
   <link name="base_footprint"/>
   <joint name="base_joint" type="fixed">
@@ -13,16 +16,16 @@
     <visual>
       <geometry>
-        <mesh filename="package://nucobot_description/meshes/bertha/body.DAE"/>
+        <mesh filename="package://nucobot_description/meshes/pikea/body.dae"/>
       </geometry>
-      <origin xyz="0.001 0 0.05199" rpy="0 0 0"/>
+      <origin xyz="0.001 0 0.0" rpy="0 0 0"/>
     </visual>
     <collision>
       <geometry>
-        <mesh filename="package://nucobot_description/meshes/bertha/body.dae"/>
+        <mesh filename="package://nucobot_description/meshes/pikea/body.dae"/>
       </geometry>
-      <origin xyz="0.0 0 0.05949" rpy="0 0 0"/>
+      <origin xyz="0.0 0 0.0" rpy="0 0 0"/>
     </collision>
     <inertial>
-      <origin xyz="0.01 0 0"/>
+      <origin xyz="0.0 0 0"/>
       <mass value="2.4"/>
       <inertia ixx="0.019995" ixy="0.0" ixz="0.0"
@@ -34,5 +37,5 @@
     <parent link="base_link"/>
     <child link="wheel_left_link"/>
-    <origin xyz="0.00 ${0.23/2} 0.0250" rpy="${-M_PI/2} 0 0"/>
+    <origin xyz="${WHEEL_SEP/2} ${WHEEL_SHIFT} ${WHEEL_HGT}" rpy="${M_PI/2} 0 0"/>
     <axis xyz="0 0 1"/>
   </joint>
@@ -40,5 +43,5 @@
     <visual>
       <geometry>
-        <cylinder length="0.0206" radius="0.0352"/>
+        <mesh filename="package://nucobot_description/meshes/pikea/wheel.dae"/>
       </geometry>
       <origin xyz="0 0 0" rpy="0 0 0"/>
@@ -46,5 +49,5 @@
     <collision>
       <geometry>
-        <cylinder length="0.0206" radius="0.0352"/>
+        <mesh filename="package://nucobot_description/meshes/pikea/wheel.dae"/>
       </geometry>
       <origin rpy="0 0 0" xyz="0 0 0"/>
@@ -61,5 +64,5 @@
     <parent link="base_link"/>
     <child link="wheel_right_link"/>
-    <origin xyz="0.00 -${0.23/2} 0.0250" rpy="${-M_PI/2} 0 0"/>
+    <origin xyz="-${WHEEL_SEP/2} ${WHEEL_SHIFT} ${WHEEL_HGT}" rpy="${-M_PI/2} 0 0"/>
     <axis xyz="0 0 1"/>
   </joint>
@@ -67,5 +70,5 @@
     <visual>
       <geometry>
-        <cylinder length="0.0206" radius="0.0350"/>
+        <mesh filename="package://nucobot_description/meshes/pikea/wheel.dae"/>
       </geometry>
       <origin xyz="0 0 0" rpy="0 0 0"/>
@@ -73,5 +76,5 @@
     <collision>
       <geometry>
-        <cylinder length="0.0206" radius="0.0350"/>
+        <mesh filename="package://nucobot_description/meshes/pikea/wheel.dae"/>
       </geometry>
       <origin rpy="0 0 0" xyz="0 0 0"/>
@@ -85,33 +88,19 @@
     </inertial>
   </link>
-  <joint name="caster_front_joint" type="fixed">
+  <joint name="wheel_front_joint" type="fixed">
     <parent link="base_link"/>
-    <child link="caster_front_link"/>
-    <origin xyz="0.115 0.0 0.007" rpy="${-M_PI/2} 0 0"/>
+    <child link="wheel_front_link"/>
+    <origin xyz="0 ${-WHEEL_SHIFT} ${WHEEL_HGT}" rpy="${M_PI/2} 0 0"/>
   </joint>
-  <link name="caster_front_link">
+  <link name="wheel_front_link">
+    <visual>
+      <geometry>
+        <mesh filename="package://nucobot_description/meshes/pikea/wheel.dae"/>
+      </geometry>
+      <origin xyz="0 0 0" rpy="0 0 0"/>
+    </visual>
     <collision>
       <geometry>
-        <cylinder length="0.0176" radius="0.017"/>
-      </geometry>
-      <origin rpy="0 0 0" xyz="0 0 0"/>
-    </collision>
-    <inertial>
-      <mass value="0.01" />
-      <origin xyz="0 0 0" />
-      <inertia ixx="0.001" ixy="0.0" ixz="0.0"
-               iyy="0.001" iyz="0.0"
-               izz="0.001" />
-    </inertial>
-  </link>
-  <joint name="caster_back_joint" type="fixed">
-    <parent link="base_link"/>
-    <child link="caster_back_link"/>
-    <origin xyz="-0.135 0.0 0.009" rpy="${-M_PI/2} 0 0"/>
-  </joint>
-  <link name="caster_back_link">
-    <collision>
-      <geometry>
-        <cylinder length="0.0176" radius="0.017"/>
+        <mesh filename="package://nucobot_description/meshes/pikea/wheel.dae"/>
       </geometry>
       <origin rpy="0 0 0" xyz="0 0 0"/>
@@ -141,13 +130,5 @@
     <maxVel>1.0</maxVel>
   </gazebo>
-  <gazebo reference="caster_front_link">
-    <mu1>0.0</mu1>
-    <mu2>0.0</mu2>
-    <kp>1000000.0</kp>
-    <kd>100.0</kd>
-    <minDepth>0.001</minDepth>
-    <maxVel>1.0</maxVel>
-  </gazebo>
-  <gazebo reference="caster_back_link">
+  <gazebo reference="wheel_front_link">
     <mu1>0.0</mu1>
     <mu2>0.0</mu2>
@@ -163,22 +144,17 @@
       <leftJoint>wheel_right_joint</leftJoint>
       <rightJoint>wheel_left_joint</rightJoint>
-      <wheelSeparation>0.230</wheelSeparation>
-      <wheelDiameter>0.070</wheelDiameter>
+      <wheelSeparation>${WHEEL_SEP}</wheelSeparation>
+      <wheelDiameter>${WHEEL_DIA}</wheelDiameter>
       <torque>20</torque>
+      <wheelTorque>20</wheelTorque>
+      <wheelAcceleration>0</wheelAcceleration>
       <commandTopic>cmd_vel</commandTopic>
       <odometryTopic>odom</odometryTopic>
       <odometryFrame>odom</odometryFrame>
+      <publishWheelTF>false</publishWheelTF>
+      <publishWheelJointState>false</publishWheelJointState>
       <robotBaseFrame>base_footprint</robotBaseFrame>
+      <rosDebugLevel>na</rosDebugLevel>
     </plugin>
   </gazebo>
-  <!-- Kinect -->
-  <xacro:include filename="$(find nucobot_description)/urdf/sensors/kinect_camera.urdf.xacro" />
-  <xacro:kinect_camera name="kinect" parent="base_link">
-    <origin xyz="${RADIUS/2} 0 ${0.3/2}" rpy="0.0 0.0 0.0"/>
-  </xacro:kinect_camera>
-  <!-- Generic camera
-  <xacro:include filename="$(find nucobot_description)/urdf/sensors/generic_camera.urdf.xacro" />
-  <xacro:generic_camera name="generic_camera" parent="base_link" ros_topic="/sensors/generic_camera/image" cam_info_topic="/sensors/generic_camera/camera_info" update_rate="15" res_x="320" res_y="240" image_format="L8" hfov="75">
-    <origin xyz="${base_x_size/2-camera_link/2} 0 ${base_z_size/2 + camera_link/2}" rpy="0 0 3.14"/>
-  </xacro:generic_camera>-->
 </robot>

Commit message: fixed pikea's inertia

File: src/nucobot_simulator/nucobot_description/urdf/pikea/pikea.urdf.xacro (robot description, xacro)
@@ -27,5 +27,5 @@
     </collision>
     <inertial>
-      <origin xyz="0.0 0 0"/>
+      <origin xyz="0 0 ${WHEEL_HGT}"/>
       <mass value="2.4"/>
       <inertia ixx="0.019995" ixy="0.0" ixz="0.0"
@@ -38,5 +38,5 @@
     <child link="wheel_left_link"/>
     <origin xyz="${WHEEL_SEP/2} ${WHEEL_SHIFT} ${WHEEL_HGT}" rpy="${M_PI/2} 0 0"/>
-    <axis xyz="0 0 1"/>
+    <axis xyz="1 0 0"/>
   </joint>
   <link name="wheel_left_link">
@@ -65,5 +65,5 @@
     <child link="wheel_right_link"/>
     <origin xyz="-${WHEEL_SEP/2} ${WHEEL_SHIFT} ${WHEEL_HGT}" rpy="${-M_PI/2} 0 0"/>
-    <axis xyz="0 0 1"/>
+    <axis xyz="1 0 0"/>
   </joint>
   <link name="wheel_right_link">
