Commit message: cahnged configs for robot models

File: src/nucobot_simulator/nucobot_description/bertha/urdf/bertha.urdf.xacro (robot description, xacro)
@@ -1,5 +1,5 @@
 <?xml version="1.0"?>
 <robot name="bertha" xmlns:xacro="http://www.ros.org/wiki/xacro">
-  <xacro:include filename="$(find nucobot_description)/urdf/materials.xacro" />
+  <xacro:include filename="$(find nucobot_description)/bertha/urdf/materials.xacro" />
   <property name="M_PI" value="3.1415926535897931" />
   <property name="RADIUS" value="0.15" />
@@ -13,5 +13,5 @@
     <visual>
       <geometry>
-        <mesh filename="package://nucobot_description/meshes/bertha/body.DAE"/>
+        <mesh filename="package://nucobot_description/bertha/meshes/body.dae"/>
       </geometry>
       <origin xyz="0.001 0 0.05199" rpy="0 0 0"/>
@@ -19,5 +19,5 @@
     <collision>
       <geometry>
-        <mesh filename="package://nucobot_description/meshes/bertha/body.dae"/>
+        <mesh filename="package://nucobot_description/bertha/meshes/body.dae"/>
       </geometry>
       <origin xyz="0.0 0 0.05949" rpy="0 0 0"/>
@@ -173,10 +173,10 @@
   </gazebo>
   <!-- Kinect -->
-  <xacro:include filename="$(find nucobot_description)/urdf/sensors/kinect_camera.urdf.xacro" />
+  <xacro:include filename="$(find nucobot_description)/bertha/urdf/kinect_camera.urdf.xacro" />
   <xacro:kinect_camera name="kinect" parent="base_link">
     <origin xyz="${RADIUS/2} 0 ${0.3/2}" rpy="0.0 0.0 0.0"/>
   </xacro:kinect_camera>
   <!-- Generic camera
-  <xacro:include filename="$(find nucobot_description)/urdf/sensors/generic_camera.urdf.xacro" />
+  <xacro:include filename="$(find nucobot_description)/bertha/urdf/generic_camera.urdf.xacro" />
   <xacro:generic_camera name="generic_camera" parent="base_link" ros_topic="/sensors/generic_camera/image" cam_info_topic="/sensors/generic_camera/camera_info" update_rate="15" res_x="320" res_y="240" image_format="L8" hfov="75">
     <origin xyz="${base_x_size/2-camera_link/2} 0 ${base_z_size/2 + camera_link/2}" rpy="0 0 3.14"/>

File: src/nucobot_simulator/nucobot_description/lisa/urdf/kinect_camera.urdf.xacro (robot description, xacro)
@@ -13,5 +13,5 @@
           <origin xyz="0 0 0" rpy="0 0 0" />
           <geometry>
-            <mesh filename="package://nucobot_description/bertha/meshes/kinect_camera_simple.dae"/>
+            <mesh filename="package://nucobot_description/lisa/meshes/kinect_camera_simple.dae"/>
           </geometry>
         </visual>
@@ -19,5 +19,5 @@
           <origin xyz="0 0 0" rpy="0 0 0" />
           <geometry>
-            <mesh filename="package://nucobot_description/bertha/meshes/kinect_camera_simple.dae"/>
+            <mesh filename="package://nucobot_description/lisa/meshes/kinect_camera_simple.dae"/>
           </geometry>
         </collision>

File: src/nucobot_simulator/nucobot_description/lisa/urdf/lisa.urdf.xacro (robot description, xacro)
@@ -1,5 +1,5 @@
 <?xml version="1.0"?>
-<robot name="test_base_kinect" xmlns:xacro="http://www.ros.org/wiki/xacro">
-  <xacro:include filename="$(find nucobot_description)/urdf/materials.xacro" />
+<robot name="lisa" xmlns:xacro="http://www.ros.org/wiki/xacro">
+  <xacro:include filename="$(find nucobot_description)/lisa/urdf/materials.xacro" />
   <property name="M_PI" value="3.1415926535897931" />
   <link name="base_footprint"/>
@@ -170,10 +170,10 @@
   </gazebo>
   <!-- Kinect -->
-  <xacro:include filename="$(find nucobot_description)/urdf/sensors/kinect_camera.urdf.xacro" />
+  <xacro:include filename="$(find nucobot_description)/lisa/urdf/kinect_camera.urdf.xacro" />
   <xacro:kinect_camera name="kinect" parent="base_link">
     <origin xyz="${0.178/2} 0 ${0.3/2}" rpy="0.0 0.0 0.0"/>
   </xacro:kinect_camera>
   <!-- Generic camera
-  <xacro:include filename="$(find nucobot_description)/urdf/sensors/generic_camera.urdf.xacro" />
+  <xacro:include filename="$(find nucobot_description)/lisa/urdf/generic_camera.urdf.xacro" />
   <xacro:generic_camera name="generic_camera" parent="base_link" ros_topic="/sensors/generic_camera/image" cam_info_topic="/sensors/generic_camera/camera_info" update_rate="15" res_x="320" res_y="240" image_format="L8" hfov="75">
     <origin xyz="${base_x_size/2-camera_link/2} 0 ${base_z_size/2 + camera_link/2}" rpy="0 0 3.14"/>

File: src/nucobot_simulator/nucobot_description/pikea/urdf/pikea.urdf.xacro (robot description, xacro)
@@ -1,5 +1,5 @@
 <?xml version="1.0"?>
 <robot name="pikea" xmlns:xacro="http://www.ros.org/wiki/xacro">
-  <xacro:include filename="$(find nucobot_description)/urdf/materials.xacro" />
+  <xacro:include filename="$(find nucobot_description)/pikea/urdf/materials.xacro" />
   <property name="M_PI" value="3.1415926535897931" />
   <property name="WHEEL_SEP" value="0.15" />
@@ -16,5 +16,5 @@
     <visual>
       <geometry>
-        <mesh filename="package://nucobot_description/meshes/pikea/body.dae"/>
+        <mesh filename="package://nucobot_description/pikea/meshes/body.dae"/>
       </geometry>
       <origin xyz="0.001 0 0.0" rpy="0 0 0"/>
@@ -22,5 +22,5 @@
     <collision>
       <geometry>
-        <mesh filename="package://nucobot_description/meshes/pikea/body.dae"/>
+        <mesh filename="package://nucobot_description/pikea/meshes/body.dae"/>
       </geometry>
       <origin xyz="0.0 0 0.0" rpy="0 0 0"/>
@@ -43,5 +43,5 @@
     <visual>
       <geometry>
-        <mesh filename="package://nucobot_description/meshes/pikea/wheel.dae"/>
+        <mesh filename="package://nucobot_description/pikea/meshes/wheel.dae"/>
       </geometry>
       <origin xyz="0 0 0" rpy="0 0 0"/>
@@ -49,5 +49,5 @@
     <collision>
       <geometry>
-        <mesh filename="package://nucobot_description/meshes/pikea/wheel.dae"/>
+        <mesh filename="package://nucobot_description/pikea/meshes/wheel.dae"/>
       </geometry>
       <origin rpy="0 0 0" xyz="0 0 0"/>
@@ -70,5 +70,5 @@
     <visual>
       <geometry>
-        <mesh filename="package://nucobot_description/meshes/pikea/wheel.dae"/>
+        <mesh filename="package://nucobot_description/pikea/meshes/wheel.dae"/>
       </geometry>
       <origin xyz="0 0 0" rpy="0 0 0"/>
@@ -76,5 +76,5 @@
     <collision>
       <geometry>
-        <mesh filename="package://nucobot_description/meshes/pikea/wheel.dae"/>
+        <mesh filename="package://nucobot_description/pikea/meshes/wheel.dae"/>
       </geometry>
       <origin rpy="0 0 0" xyz="0 0 0"/>
@@ -96,5 +96,5 @@
     <visual>
       <geometry>
-        <mesh filename="package://nucobot_description/meshes/pikea/wheel.dae"/>
+        <mesh filename="package://nucobot_description/pikea/meshes/wheel.dae"/>
       </geometry>
       <origin xyz="0 0 0" rpy="0 0 0"/>
@@ -102,5 +102,5 @@
     <collision>
       <geometry>
-        <mesh filename="package://nucobot_description/meshes/pikea/wheel.dae"/>
+        <mesh filename="package://nucobot_description/pikea/meshes/wheel.dae"/>
       </geometry>
       <origin rpy="0 0 0" xyz="0 0 0"/>
