Commit message: added gripper to pikea

File: src/nucobot_simulator/nucobot_description/map_objects/urdf/beacon.xacro (robot description, xacro)
@@ -6,7 +6,7 @@
   <xacro:property name="height" value="0.16" />
   <!-- Import all Gazebo-customization elements, including Gazebo colors -->
-  <xacro:include filename="$(find nucobot_description)/urdf/beacon/beacon.gazebo" />
+  <xacro:include filename="$(find nucobot_description)/map_objects/urdf/beacon.gazebo" />
   <!-- Import Rviz colors -->
-  <xacro:include filename="$(find nucobot_description)/urdf/materials.xacro" />
+  <xacro:include filename="$(find nucobot_description)/map_objects/urdf/materials.xacro" />
   <!-- Camera -->
   <link name="beacon_$(arg prefix)_base_link">

File: src/nucobot_simulator/nucobot_description/map_objects/urdf/cup.xacro (robot description, xacro)
@@ -10,5 +10,5 @@
       <origin xyz="0 0 0" rpy="0 0 0"/>
       <geometry>
-        <mesh filename="package://nucobot_description/meshes/toys/cup.dae"/>
+        <mesh filename="package://nucobot_description/map_objects/meshes/cup.dae"/>
       </geometry>
     </collision>
@@ -16,5 +16,5 @@
       <origin xyz="0 0 0" rpy="0 0 0"/>
       <geometry>
-        <mesh filename="package://nucobot_description/meshes/toys/cup.dae"/>
+        <mesh filename="package://nucobot_description/map_objects/meshes/cup.dae"/>
       </geometry>
     </visual>

File: src/nucobot_simulator/nucobot_description/map_objects/urdf/cylinder.xacro (robot description, xacro)
@@ -10,5 +10,5 @@
       <origin xyz="0 0 0" rpy="0 0 0"/>
       <geometry>
-        <mesh filename="package://nucobot_description/meshes/toys/cylinder.dae"/>
+        <mesh filename="package://nucobot_description/map_objects/meshes/cylinder.dae"/>
       </geometry>
     </collision>
@@ -16,5 +16,5 @@
       <origin xyz="0 0 0" rpy="0 0 0"/>
       <geometry>
-        <mesh filename="package://nucobot_description/meshes/toys/cylinder.dae"/>
+        <mesh filename="package://nucobot_description/map_objects/meshes/cylinder.dae"/>
       </geometry>
     </visual>

File: src/nucobot_simulator/nucobot_description/map_objects/urdf/pop_corn_ball.xacro (robot description, xacro)
@@ -9,5 +9,5 @@
       <origin xyz="0 0 0" rpy="0 0 0"/>
       <geometry>
-        <mesh filename="package://nucobot_description/meshes/toys/pop_corn_ball.dae"/>
+        <mesh filename="package://nucobot_description/map_objects/meshes/pop_corn_ball.dae"/>
       </geometry>
     </collision>
@@ -15,5 +15,5 @@
       <origin xyz="0 0 0" rpy="0 0 0"/>
       <geometry>
-        <mesh filename="package://nucobot_description/meshes/toys/pop_corn_ball.dae"/>
+        <mesh filename="package://nucobot_description/map_objects/meshes/pop_corn_ball.dae"/>
       </geometry>
     </visual>

File: src/nucobot_simulator/nucobot_description/map_objects/urdf/tennis_ball.xacro (robot description, xacro)
@@ -9,5 +9,5 @@
       <origin xyz="0 0 0" rpy="0 0 0"/>
       <geometry>
-        <mesh filename="package://nucobot_description/meshes/toys/tennis_ball.dae"/>
+        <mesh filename="package://nucobot_description/map_objects/meshes/tennis_ball.dae"/>
       </geometry>
     </collision>
@@ -15,5 +15,5 @@
       <origin xyz="0 0 0" rpy="0 0 0"/>
       <geometry>
-        <mesh filename="package://nucobot_description/meshes/toys/tennis_ball.dae"/>
+        <mesh filename="package://nucobot_description/map_objects/meshes/tennis_ball.dae"/>
       </geometry>
     </visual>

File: src/nucobot_simulator/nucobot_description/pikea/urdf/pikea_gripper.urdf.xacro (robot description, xacro)
@@ -11,13 +11,15 @@
     <visual>
       <geometry>
-        <mesh filename="package://nucobot_description/pikea/meshes/left_hand_outer.dae"/>
+        <mesh filename="package://nucobot_description/pikea/meshes/finger_visual.STL"
+              scale="0.001 0.001 0.001"/>
       </geometry>
-      <origin xyz="0 0 0" rpy="0 0 0"/>
+      <origin xyz="0.0 0.08 -0.007" rpy="${pi/2} 0 0"/>
     </visual>
     <collision>
       <geometry>
-        <mesh filename="package://nucobot_description/pikea/meshes/left_hand_outer.dae"/>
+        <mesh filename="package://nucobot_description/pikea/meshes/finger_simple.STL"
+              scale="0.001 0.001 0.001"/>
       </geometry>
-      <origin xyz="0 0 0" rpy="0 0 0"/>
+      <origin xyz="0.0 0.08 -0.007" rpy="${pi/2} 0 0"/>
     </collision>
     <inertial>
@@ -60,5 +62,8 @@
   <!-- ... And two fingers -->
   <xacro:grip_finger name="${name}_left_finger" parent="${name}_link">
-     <origin xyz="0.0 0.02 0.0" rpy="0 0 0"/>
+     <origin xyz=" 0.003 0.0 0.0" rpy="0 0 0"/>
+  </xacro:grip_finger>
+  <xacro:grip_finger name="${name}_rght_finger" parent="${name}_link">
+     <origin xyz="-0.003 0.0 0.0" rpy="0 ${pi} 0"/>
   </xacro:grip_finger>
   </xacro:macro>
