Commit message: add gripper control

File: src/nucobot_simulator/nucobot_description/pikea/urdf/pikea.gazebo.xacro (robot description, xacro)
@@ -1,4 +1,10 @@
 <?xml version="1.0"?>
 <robot name="pikea" xmlns:xacro="http://ros.org/wiki/xacro">
-    <xacro:include filename="$(find nucobot_description)/pikea/urdf/pikea.urdf.xacro" />
+  <gazebo>
+    <plugin name="gazebo_ros_control" filename="libgazebo_ros_control.so">
+      <robotNamespace>/pikea</robotNamespace>
+      <robotSimType>gazebo_ros_control/DefaultRobotHWSim</robotSimType>
+    </plugin>
+  </gazebo>
+  <xacro:include filename="$(find nucobot_description)/pikea/urdf/pikea.urdf.xacro" />
 </robot>

File: src/nucobot_simulator/nucobot_description/pikea/urdf/pikea.urdf.xacro (robot description, xacro)
@@ -7,6 +7,14 @@
   <!-- Gripper(s) -->
   <xacro:include filename="$(find nucobot_description)/pikea/urdf/pikea_gripper.urdf.xacro" />
-  <xacro:gripper name="gripper_1" parent="base_link" ros_topic="gripper1">
-     <origin xyz="0.1 0.1 0.1" rpy="0 0 0"/>
+  <xacro:gripper name="gripper_1" parent="base_link">
+     <origin xyz="0.05 0.05 0.0" rpy="0 0 0"/>
   </xacro:gripper>
+  <xacro:gripper name="gripper_2" parent="base_link">
+     <origin xyz="-0.05 0.05 0.0" rpy="0 0 0"/>
+  </xacro:gripper>
+  <!-- Wheels -->
+  <xacro:include filename="$(find nucobot_description)/pikea/urdf/pikea_diff_drive.urdf.xacro" />
+  <xacro:diff_drive name="pikea_drive" parent="base_link" wheelSeparation="0.15" wheelDiameter="0.07">
+     <origin xyz="0.0 0.04 -0.08" rpy="0 0 0"/>
+  </xacro:diff_drive>
 </robot>

File: src/nucobot_simulator/nucobot_description/pikea/urdf/pikea_base.urdf.xacro (robot description, xacro)
@@ -25,4 +25,38 @@
     </inertial>
   </link>
+  <joint name="caster_joint" type="fixed">
+    <parent link="base_link"/>
+    <child link="caster_link"/>
+    <origin xyz="0 -0.04 -0.08" rpy="${pi/2} 0 0"/>
+  </joint>
+  <link name="caster_link">
+    <visual>
+      <geometry>
+        <mesh filename="package://nucobot_description/pikea/meshes/wheel.dae"/>
+      </geometry>
+      <origin xyz="0 0 0" rpy="0 0 0"/>
+    </visual>
+    <collision>
+      <geometry>
+        <mesh filename="package://nucobot_description/pikea/meshes/wheel.dae"/>
+      </geometry>
+      <origin rpy="0 0 0" xyz="0 0 0"/>
+    </collision>
+    <inertial>
+      <mass value="0.01" />
+      <origin xyz="0 0 0" />
+      <inertia ixx="0.001" ixy="0.0" ixz="0.0"
+               iyy="0.001" iyz="0.0"
+               izz="0.001" />
+    </inertial>
+  </link>
+  <gazebo reference="caster_link">
+    <mu1>0.0</mu1>
+    <mu2>0.0</mu2>
+    <kp>1000000.0</kp>
+    <kd>100.0</kd>
+    <minDepth>0.001</minDepth>
+    <maxVel>1.0</maxVel>
+  </gazebo>
   </xacro:macro>
 </robot>

File: src/nucobot_simulator/nucobot_description/pikea/urdf/pikea_gripper.urdf.xacro (robot description, xacro)
@@ -3,8 +3,10 @@
   <xacro:property name="pi" value="3.1415926535897931" />
   <xacro:macro name="grip_finger" params="name parent *origin">
-  <joint name="${name}_joint" type="fixed">
+  <joint name="${name}_joint" type="continuous">
       <xacro:insert_block name="origin" />
       <parent link="${parent}"/>
       <child link="${name}_link"/>
+      <axis xyz="0 0 1"/>
+      <dynamics damping="0.7"/>
   </joint>
   <link name="${name}_link">
@@ -25,12 +27,20 @@
     <inertial>
       <origin xyz="0 0 0"/>
-      <mass value="0.1"/>
-      <inertia ixx="0.1" ixy="0.0" ixz="0.0"
-               iyy="0.1" iyz="0.0"
-               izz="0.1" />
+      <mass value="0.01"/>
+      <inertia ixx="0.001" ixy="0.0" ixz="0.0"
+               iyy="0.001" iyz="0.0"
+               izz="0.001" />
     </inertial>
   </link>
+  <transmission name="${name}_transmission">
+    <type>transmission_interface/SimpleTransmission</type>
+    <joint name="${name}_joint"/>
+    <actuator name="${name}_servo">
+      <hardwareInterface>EffortJointInterface</hardwareInterface>
+      <mechanicalReduction>1</mechanicalReduction>
+    </actuator>
+  </transmission>
   </xacro:macro>
-  <xacro:macro name="gripper" params="name parent *origin ros_topic">
+  <xacro:macro name="gripper" params="name parent *origin">
   <!-- The gripper base -->
   <joint name="${name}_joint" type="fixed">
@@ -61,8 +71,8 @@
   </link>
   <!-- ... And two fingers -->
-  <xacro:grip_finger name="${name}_left_finger" parent="${name}_link">
+  <xacro:grip_finger name="${name}_rght_finger" parent="${name}_link">
      <origin xyz=" 0.003 0.0 0.0" rpy="0 0 0"/>
   </xacro:grip_finger>
-  <xacro:grip_finger name="${name}_rght_finger" parent="${name}_link">
+  <xacro:grip_finger name="${name}_left_finger" parent="${name}_link">
      <origin xyz="-0.003 0.0 0.0" rpy="0 ${pi} 0"/>
   </xacro:grip_finger>
