Commit message: adding a gripper to pikea

File: src/nucobot_simulator/nucobot_description/pikea/urdf/pikea.urdf.xacro (robot description, xacro)
@@ -1,160 +1,12 @@
 <?xml version="1.0"?>
-<robot name="pikea" xmlns:xacro="http://www.ros.org/wiki/xacro">
-  <xacro:include filename="$(find nucobot_description)/pikea/urdf/materials.xacro" />
-  <property name="M_PI" value="3.1415926535897931" />
-  <property name="WHEEL_SEP" value="0.15" />
-  <property name="WHEEL_DIA" value="0.07" />
-  <property name="WHEEL_HGT" value="-0.08" />
-  <property name="WHEEL_SHIFT" value="-0.02" />
-  <link name="base_footprint"/>
-  <joint name="base_joint" type="fixed">
-    <origin xyz="0 0 0.0102" rpy="0 0 0" />
-    <parent link="base_footprint"/>
-    <child link="base_link" />
-  </joint>
-  <link name="base_link">
-    <visual>
-      <geometry>
-        <mesh filename="package://nucobot_description/pikea/meshes/body.dae"/>
-      </geometry>
-      <origin xyz="0.001 0 0.0" rpy="0 0 0"/>
-    </visual>
-    <collision>
-      <geometry>
-        <mesh filename="package://nucobot_description/pikea/meshes/body.dae"/>
-      </geometry>
-      <origin xyz="0.0 0 0.0" rpy="0 0 0"/>
-    </collision>
-    <inertial>
-      <origin xyz="0 0 ${WHEEL_HGT}"/>
-      <mass value="2.4"/>
-      <inertia ixx="0.019995" ixy="0.0" ixz="0.0"
-               iyy="0.019995" iyz="0.0"
-               izz="0.03675" />
-    </inertial>
-  </link>
-  <joint name="wheel_left_joint" type="continuous">
-    <parent link="base_link"/>
-    <child link="wheel_left_link"/>
-    <origin xyz="${WHEEL_SEP/2} ${WHEEL_SHIFT} ${WHEEL_HGT}" rpy="${M_PI/2} 0 0"/>
-    <axis xyz="1 0 0"/>
-  </joint>
-  <link name="wheel_left_link">
-    <visual>
-      <geometry>
-        <mesh filename="package://nucobot_description/pikea/meshes/wheel.dae"/>
-      </geometry>
-      <origin xyz="0 0 0" rpy="0 0 0"/>
-    </visual>
-    <collision>
-      <geometry>
-        <mesh filename="package://nucobot_description/pikea/meshes/wheel.dae"/>
-      </geometry>
-      <origin rpy="0 0 0" xyz="0 0 0"/>
-    </collision>
-    <inertial>
-      <mass value="0.01" />
-      <origin xyz="0 0 0" />
-      <inertia ixx="0.001" ixy="0.0" ixz="0.0"
-               iyy="0.001" iyz="0.0"
-               izz="0.001" />
-    </inertial>
-  </link>
-  <joint name="wheel_right_joint" type="continuous">
-    <parent link="base_link"/>
-    <child link="wheel_right_link"/>
-    <origin xyz="-${WHEEL_SEP/2} ${WHEEL_SHIFT} ${WHEEL_HGT}" rpy="${-M_PI/2} 0 0"/>
-    <axis xyz="1 0 0"/>
-  </joint>
-  <link name="wheel_right_link">
-    <visual>
-      <geometry>
-        <mesh filename="package://nucobot_description/pikea/meshes/wheel.dae"/>
-      </geometry>
-      <origin xyz="0 0 0" rpy="0 0 0"/>
-    </visual>
-    <collision>
-      <geometry>
-        <mesh filename="package://nucobot_description/pikea/meshes/wheel.dae"/>
-      </geometry>
-      <origin rpy="0 0 0" xyz="0 0 0"/>
-    </collision>
-    <inertial>
-      <mass value="0.01" />
-      <origin xyz="0 0 0" />
-      <inertia ixx="0.001" ixy="0.0" ixz="0.0"
-               iyy="0.001" iyz="0.0"
-               izz="0.001" />
-    </inertial>
-  </link>
-  <joint name="wheel_front_joint" type="fixed">
-    <parent link="base_link"/>
-    <child link="wheel_front_link"/>
-    <origin xyz="0 ${-WHEEL_SHIFT} ${WHEEL_HGT}" rpy="${M_PI/2} 0 0"/>
-  </joint>
-  <link name="wheel_front_link">
-    <visual>
-      <geometry>
-        <mesh filename="package://nucobot_description/pikea/meshes/wheel.dae"/>
-      </geometry>
-      <origin xyz="0 0 0" rpy="0 0 0"/>
-    </visual>
-    <collision>
-      <geometry>
-        <mesh filename="package://nucobot_description/pikea/meshes/wheel.dae"/>
-      </geometry>
-      <origin rpy="0 0 0" xyz="0 0 0"/>
-    </collision>
-    <inertial>
-      <mass value="0.01" />
-      <origin xyz="0 0 0" />
-      <inertia ixx="0.001" ixy="0.0" ixz="0.0"
-               iyy="0.001" iyz="0.0"
-               izz="0.001" />
-    </inertial>
-  </link>
-  <gazebo reference="wheel_left_link">
-    <mu1>1.0</mu1>
-    <mu2>1.0</mu2>
-    <kp>1000000.0</kp>
-    <kd>100.0</kd>
-    <minDepth>0.001</minDepth>
-    <maxVel>1.0</maxVel>
-  </gazebo>
-  <gazebo reference="wheel_right_link">
-    <mu1>1.0</mu1>
-    <mu2>1.0</mu2>
-    <kp>1000000.0</kp>
-    <kd>100.0</kd>
-    <minDepth>0.001</minDepth>
-    <maxVel>1.0</maxVel>
-  </gazebo>
-  <gazebo reference="wheel_front_link">
-    <mu1>0.0</mu1>
-    <mu2>0.0</mu2>
-    <kp>1000000.0</kp>
-    <kd>100.0</kd>
-    <minDepth>0.001</minDepth>
-    <maxVel>1.0</maxVel>
-  </gazebo>
-  <gazebo>
-    <plugin name="differential_drive_controller" filename="libgazebo_ros_diff_drive.so">
-      <alwaysOn>true</alwaysOn>
-      <updateRate>100</updateRate>
-      <leftJoint>wheel_right_joint</leftJoint>
-      <rightJoint>wheel_left_joint</rightJoint>
-      <wheelSeparation>${WHEEL_SEP}</wheelSeparation>
-      <wheelDiameter>${WHEEL_DIA}</wheelDiameter>
-      <torque>20</torque>
-      <wheelTorque>20</wheelTorque>
-      <wheelAcceleration>0</wheelAcceleration>
-      <commandTopic>cmd_vel</commandTopic>
-      <odometryTopic>odom</odometryTopic>
-      <odometryFrame>odom</odometryFrame>
-      <publishWheelTF>false</publishWheelTF>
-      <publishWheelJointState>false</publishWheelJointState>
-      <robotBaseFrame>base_footprint</robotBaseFrame>
-      <rosDebugLevel>na</rosDebugLevel>
-    </plugin>
-  </gazebo>
+<robot name="pikea" xmlns:xacro="http://ros.org/wiki/xacro">
+  <xacro:property name="pi" value="3.1415926535897931" />
+  <!-- The body -->
+  <xacro:include filename="$(find nucobot_description)/pikea/urdf/pikea_base.urdf.xacro" />
+  <xacro:pikea_base_macro wheel_h="-0.08"/>
+  <!-- Gripper(s) -->
+  <xacro:include filename="$(find nucobot_description)/pikea/urdf/pikea_gripper.urdf.xacro" />
+  <xacro:gripper name="gripper_1" parent="base_link" ros_topic="gripper1">
+     <origin xyz="0.1 0.1 0.1" rpy="0 0 0"/>
+  </xacro:gripper>
 </robot>

Commit message: add manual control package

File: src/nucobot_simulator/nucobot_description/pikea/urdf/pikea.urdf.xacro (robot description, xacro)
@@ -16,5 +16,5 @@
   <xacro:include filename="$(find nucobot_description)/pikea/urdf/pikea_diff_drive.urdf.xacro" />
   <xacro:diff_drive name="pikea_drive" parent="base_link" wheelSeparation="0.15" wheelDiameter="0.07">
-     <origin xyz="0.0 0.04 -0.08" rpy="0 0 0"/>
+     <origin xyz="0.0 0.04 -0.08" rpy="0 0 ${pi}"/>
   </xacro:diff_drive>
 </robot>

File: src/nucobot_simulator/nucobot_description/pikea/urdf/pikea_base.urdf.xacro (robot description, xacro)
@@ -19,8 +19,8 @@
     <inertial>
       <origin xyz="0 0 ${wheel_h}"/>
-      <mass value="2.4"/>
-      <inertia ixx="0.019995" ixy="0.0" ixz="0.0"
-               iyy="0.019995" iyz="0.0"
-               izz="0.03675" />
+      <mass value="3.4"/>
+      <inertia ixx="0.57" ixy="0.0" ixz="0.0"
+               iyy="0.57" iyz="0.0"
+               izz="0.57" />
     </inertial>
   </link>

File: src/nucobot_simulator/nucobot_description/pikea/urdf/pikea_gripper.urdf.xacro (robot description, xacro)
@@ -33,4 +33,12 @@
     </inertial>
   </link>
+  <gazebo reference="${name}_link">
+    <mu1>1.0</mu1>
+    <mu2>1.0</mu2>
+    <kp>1000000.0</kp>
+    <kd>100.0</kd>
+    <minDepth>0.001</minDepth>
+    <maxVel>1.0</maxVel>
+  </gazebo>
   <transmission name="${name}_transmission">
     <type>transmission_interface/SimpleTransmission</type>

Commit message: checked gripper functionality

File: src/nucobot_simulator/nucobot_description/pikea/urdf/pikea.urdf.xacro (robot description, xacro)
@@ -8,8 +8,8 @@
   <xacro:include filename="$(find nucobot_description)/pikea/urdf/pikea_gripper.urdf.xacro" />
   <xacro:gripper name="gripper_1" parent="base_link">
-     <origin xyz="0.05 0.05 0.0" rpy="0 0 0"/>
+     <origin xyz=" 0.05 0.05 -0.02" rpy="0 0 0"/>
   </xacro:gripper>
   <xacro:gripper name="gripper_2" parent="base_link">
-     <origin xyz="-0.05 0.05 0.0" rpy="0 0 0"/>
+     <origin xyz="-0.05 0.05 -0.02" rpy="0 0 0"/>
   </xacro:gripper>
   <!-- Wheels -->

File: src/nucobot_simulator/nucobot_description/pikea/urdf/pikea_base.urdf.xacro (robot description, xacro)
@@ -4,4 +4,18 @@
   <!-- Main link -->
   <xacro:macro name="pikea_base_macro" params="wheel_h">
+  <joint name="base_to_footprint_joint" type="fixed">
+    <parent link="base_link"/>
+    <child link="base_footprint"/>
+    <origin xyz="0 0.0 ${wheel_h}" rpy="0 0 0"/>
+  </joint>
+  <link name="base_footprint">
+    <inertial>
+      <mass value="0.001" />
+      <origin xyz="0 0 0" />
+      <inertia ixx="0.0001" ixy="0.0" ixz="0.0"
+               iyy="0.0001" iyz="0.0"
+               izz="0.0001" />
+    </inertial>
+  </link>
   <link name="base_link">
     <visual>
@@ -19,8 +33,8 @@
     <inertial>
       <origin xyz="0 0 ${wheel_h}"/>
-      <mass value="3.4"/>
-      <inertia ixx="0.57" ixy="0.0" ixz="0.0"
-               iyy="0.57" iyz="0.0"
-               izz="0.57" />
+      <mass value="2.4"/>
+      <inertia ixx="0.27" ixy="0.0" ixz="0.0"
+               iyy="0.27" iyz="0.0"
+               izz="0.27" />
     </inertial>
   </link>
@@ -28,5 +42,5 @@
     <parent link="base_link"/>
     <child link="caster_link"/>
-    <origin xyz="0 -0.04 -0.08" rpy="${pi/2} 0 0"/>
+    <origin xyz="0 -0.04 ${wheel_h}" rpy="${pi/2} 0 0"/>
   </joint>
   <link name="caster_link">

File: src/nucobot_simulator/nucobot_description/pikea/urdf/pikea_diff_drive.urdf.xacro (robot description, xacro)
@@ -76,6 +76,6 @@
       <odometryTopic>odom</odometryTopic>
       <odometryFrame>odom</odometryFrame>
-      <publishWheelTF>false</publishWheelTF>
-      <publishWheelJointState>false</publishWheelJointState>
+      <publishWheelTF>true</publishWheelTF>
+      <publishWheelJointState>true</publishWheelJointState>
       <robotBaseFrame>${parent}</robotBaseFrame>
       <rosDebugLevel>na</rosDebugLevel>
